File: kicad/v06ckeyboard/v06ckeyboard.kicad_pcb (KiCad board)
At the start: 2 copper layers, 150 x 56 mm, 114 parts, among them J1 Conn_01x24, J2 SH1.0-7, J3 SH1.0-7, SW100_ВВОД1 SKPMAME010, SW101_СБР1 SKPMAME010, SW102_БЛК1 SKPMAME010, SW103_СС1 SKPMAME010, SW104_УС1 SKPMAME010, SW105_РУС/LAT1 SKPMAME010, SW10_1 SKPMAME010, SW11_9 SKPMAME010, SW12_А1 SKPMAME010, SW13_И1 SKPMAME010, SW14_Я1 SKPMAME010, SW15_Ы1 SKPMAME010, SW16_СТР1 SKPMAME010, SW17_ВК1 SKPMAME010, SW18_2 SKPMAME010, SW19_:1 SKPMAME010, SW1_ТАБ1 SKPMAME010, SW20_Б1 SKPMAME010, SW21_Й1 SKPMAME010, SW22_Р1 SKPMAME010, SW23_З1 SKPMAME010, SW24_AP2 SKPMAME010, SW25_ЗБ1 SKPMAME010, SW26_3 SKPMAME010, SW27_;1 SKPMAME010, SW28_Ц1 SKPMAME010, SW29_К1 SKPMAME010, SW2_0 SKPMAME010, SW30_С1 SKPMAME010, SW31_Ш1 SKPMAME010, SW32_F1 SKPMAME010, SW33_LT1 SKPMAME010, SW34_4 SKPMAME010, SW35 SKPMAME010, SW36_Д1 SKPMAME010, SW37_Л1 SKPMAME010, SW38_Т1 SKPMAME010, SW39_Э1 SKPMAME010, SW3_8 SKPMAME010, SW40_F2 SKPMAME010, SW41_UP1 SKPMAME010, SW42_5 SKPMAME010, SW43_-=1 SKPMAME010, SW44_E1 SKPMAME010, SW45_М1 SKPMAME010, SW46_У1 SKPMAME010, SW47_Щ1 SKPMAME010, SW48_F3 SKPMAME010, SW49_RT1 SKPMAME010, SW4_Ю1 SKPMAME010, SW50_6 SKPMAME010, SW51 SKPMAME010, SW52_Ф1 SKPMAME010, SW53_Н1 SKPMAME010, SW54_Ж1 SKPMAME010, SW55_Ч1 SKPMAME010, SW56_F4 SKPMAME010, SW57_DN1 SKPMAME010, SW58_7 SKPMAME010, SW59_/1 SKPMAME010, SW5_Х1 SKPMAME010, SW60_Г1 SKPMAME010, SW61_О1 SKPMAME010, SW62_В1 SKPMAME010, SW63_SPC1 SKPMAME010, SW63_SPC2 SKPMAME010, SW64_F5 SKPMAME010, SW6_П1 SKPMAME010, SW7_Ь1 SKPMAME010, SW8_HOME1 SKPMAME010, SW9_ПС1 SKPMAME010, U1 Pico

Commit message: readme lala
Parts:
- added D12: BAT54S, Package_TO_SOT_SMD:SOT-23, F.Cu at (229.0, 138.8)
Connections:
- U1 pad 39: /VSYS -> /VSYSx
Routing:
- net /VSYS: track 118.5 -> 45.0 mm, vias 2 -> 1
- net /VSYSx: track 0.00 -> 72.3 mm, vias 0 -> 1
Changed lines of the file:
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@@
   (net 56 "unconnected-(J2-Pin_6-Pad6)")
   (net 57 "/VSYS")
+  (net 58 "unconnected-(D12-A-Pad1)")
+  (net 59 "/VSYSx")
   (footprint "SKPM_Alps:SKPM" locked (layer "F.Cu")
     (at 132 100)
@@
     )
   )
+  (footprint "Package_TO_SOT_SMD:SOT-23" (layer "F.Cu")
+    (at 228.9625 138.75 180)
+    (descr "SOT, 3 Pin (https://www.jedec.org/system/files/docs/to-236h.pdf variant AB), generated with kicad-footprint-generator ipc_gullwing_generator.py")
+    (tags "SOT TO_SOT_SMD")
+    (property "Sheetfile" "v06ckeyboard.kicad_sch")
+    (property "Sheetname" "")
+    (property "ki_description" "Vr 30V, If 200mA, Dual schottky barrier diode, in series, SOT-323")
+    (property "ki_keywords" "schottky diode")
+    (attr smd)
+    (fp_text reference "D12" (at 3.4625 -0.05) (layer "F.SilkS")
+        (effects (font (size 1 1) (thickness 0.15)))
+    )
+    (fp_text value "BAT54S" (at 0 2.4) (layer "F.Fab")
+        (effects (font (size 1 1) (thickness 0.15)))
+    )
+    (fp_text user "${REFERENCE}" (at 0 0) (layer "F.Fab")
+        (effects (font (size 0.32 0.32) (thickness 0.05)))
+    )
+    (fp_line (start 0 -1.56) (end -1.675 -1.56)
+      (stroke (width 0.12) (type solid)) (layer "F.SilkS"))
+    (fp_line (start 0 -1.56) (end 0.65 -1.56)
+      (stroke (width 0.12) (type solid)) (layer "F.SilkS"))
+    (fp_line (start 0 1.56) (end -0.65 1.56)
+      (stroke (width 0.12) (type solid)) (layer "F.SilkS"))
+    (fp_line (start 0 1.56) (end 0.65 1.56)
+      (stroke (width 0.12) (type solid)) (layer "F.SilkS"))
+    (fp_line (start -1.92 -1.7) (end -1.92 1.7)
+      (stroke (width 0.05) (type solid)) (layer "F.CrtYd"))
+    (fp_line (start -1.92 1.7) (end 1.92 1.7)
+      (stroke (width 0.05) (type solid)) (layer "F.CrtYd"))
+    (fp_line (start 1.92 -1.7) (end -1.92 -1.7)
+      (stroke (width 0.05) (type solid)) (layer "F.CrtYd"))
+    (fp_line (start 1.92 1.7) (end 1.92 -1.7)
+      (stroke (width 0.05) (type solid)) (layer "F.CrtYd"))
+    (fp_line (start -0.65 -1.125) (end -0.325 -1.45)
+      (stroke (width 0.1) (type solid)) (layer "F.Fab"))
+    (fp_line (start -0.65 1.45) (end -0.65 -1.125)
+      (stroke (width 0.1) (type solid)) (layer "F.Fab"))
+    (fp_line (start -0.325 -1.45) (end 0.65 -1.45)
+      (stroke (width 0.1) (type solid)) (layer "F.Fab"))
+    (fp_line (start 0.65 -1.45) (end 0.65 1.45)
+      (stroke (width 0.1) (type solid)) (layer "F.Fab"))
+    (fp_line (start 0.65 1.45) (end -0.65 1.45)
+      (stroke (width 0.1) (type solid)) (layer "F.Fab"))
+    (pad "1" smd roundrect (at -0.9375 -0.95 180) (size 1.475 0.6) (layers "F.Cu" "F.Paste" "F.Mask") (roundrect_rratio 0.25)
+      (net 58 "unconnected-(D12-A-Pad1)") (pinfunction "A") (pintype "passive+no_connect"))
+    (pad "2" smd roundrect (at -0.9375 0.95 180) (size 1.475 0.6) (layers "F.Cu" "F.Paste" "F.Mask") (roundrect_rratio 0.25)
+      (net 59 "/VSYSx") (pinfunction "K") (pintype "passive"))
+    (pad "3" smd roundrect (at 0.9375 0 180) (size 1.475 0.6) (layers "F.Cu" "F.Paste" "F.Mask") (roundrect_rratio 0.25)
+      (net 57 "/VSYS") (pinfunction "COM") (pintype "passive"))
+    (model "${KICAD6_3DMODEL_DIR}/Package_TO_SOT_SMD.3dshapes/SOT-23.wrl"
+      (offset (xyz 0 0 0))
+      (scale (xyz 1 1 1))
+      (rotate (xyz 0 0 0))
+    )
+  )
   (footprint "Resistor_SMD:R_0603_1608Metric" (layer "F.Cu")
     (at 174 94 -90)
@@
       (net 19 "GND") (pinfunction "GND") (pintype "bidirectional"))
     (pad "39" smd rect (at 8.89 21.59 180) (size 3.5 1.7) (drill (offset 0.9 0)) (layers "B.Cu" "B.Mask")
-      (net 57 "/VSYS") (pinfunction "VSYS") (pintype "power_in"))
+      (net 59 "/VSYSx") (pinfunction "VSYS") (pintype "power_in"))
     (pad "40" smd rect (at 8.89 24.13 180) (size 3.5 1.7) (drill (offset 0.9 0)) (layers "B.Cu" "B.Mask")
       (net 51 "unconnected-(U1-VBUS-Pad40)") (pinfunction "VBUS") (pintype "power_in"))
@@
   (segment (start 191.3 135.625) (end 191.3 136.071751) (width 0.25) (layer "B.Cu") (net 47))
   (segment (start 211.665 137.735) (end 211.665 136.535) (width 0.25) (layer "B.Cu") (net 47))
-  (segment (start 215.38 137.4) (end 231.9 137.4) (width 0.5) (layer "F.Cu") (net 57))
-  (segment (start 234.1 93.1) (end 229.23 88.23) (width 0.5) (layer "F.Cu") (net 57))
   (segment (start 212.98 139.8) (end 189 139.8) (width 0.5) (layer "F.Cu") (net 57))
-  (segment (start 234.1 135.2) (end 234.1 93.1) (width 0.5) (layer "F.Cu") (net 57))
-  (segment (start 211.67 88.23) (end 211.3 88.6) (width 0.5) (layer "F.Cu") (net 57))
   (segment (start 189 139.8) (end 188.3 139.1) (width 0.5) (layer "F.Cu") (net 57))
-  (segment (start 229.23 88.23) (end 211.67 88.23) (width 0.5) (layer "F.Cu") (net 57))
-  (segment (start 231.9 137.4) (end 234.1 135.2) (width 0.5) (layer "F.Cu") (net 57))
+  (segment (start 228.025 138.75) (end 216.73 138.75) (width 0.5) (layer "F.Cu") (net 57))
   (segment (start 215.38 137.4) (end 212.98 139.8) (width 0.5) (layer "F.Cu") (net 57))
+  (segment (start 216.73 138.75) (end 215.38 137.4) (width 0.5) (layer "F.Cu") (net 57))
   (segment (start 188.3 139.1) (end 188.3 138) (width 0.5) (layer "F.Cu") (net 57))
   (via (at 188.3 138) (size 0.8) (drill 0.4) (layers "F.Cu" "B.Cu") (net 57))
-  (via (at 211.3 88.6) (size 0.8) (drill 0.4) (layers "F.Cu" "B.Cu") (net 57))
   (segment (start 188.3 138) (end 188.3 135.625) (width 0.5) (layer "B.Cu") (net 57))
+  (segment (start 229.9 137.8) (end 231.5 137.8) (width 0.5) (layer "F.Cu") (net 59))
+  (segment (start 229.23 88.23) (end 211.67 88.23) (width 0.5) (layer "F.Cu") (net 59))
+  (segment (start 211.67 88.23) (end 211.3 88.6) (width 0.5) (layer "F.Cu") (net 59))
+  (segment (start 231.5 137.8) (end 234.1 135.2) (width 0.5) (layer "F.Cu") (net 59))
+  (segment (start 234.1 93.1) (end 229.23 88.23) (width 0.5) (layer "F.Cu") (net 59))
+  (segment (start 234.1 135.2) (end 234.1 93.1) (width 0.5) (layer "F.Cu") (net 59))
+  (via (at 211.3 88.6) (size 0.8) (drill 0.4) (layers "F.Cu" "B.Cu") (net 59))
 )
