File: kicad/v06ckeyboard/v06ckeyboard.kicad_sch (KiCad schematic)
At the start: 114 parts, among them J1 Conn_01x24, J2 SH1.0-7, J3 SH1.0-7, SW100_ВВОД1 SKPMAME010, SW101_СБР1 SKPMAME010, SW102_БЛК1 SKPMAME010, SW103_СС1 SKPMAME010, SW104_УС1 SKPMAME010, SW105_РУС/LAT1 SKPMAME010, SW10_1 SKPMAME010, SW11_9 SKPMAME010, SW12_А1 SKPMAME010, SW13_И1 SKPMAME010, SW14_Я1 SKPMAME010, SW15_Ы1 SKPMAME010, SW16_СТР1 SKPMAME010, SW17_ВК1 SKPMAME010, SW18_2 SKPMAME010, SW19_:1 SKPMAME010, SW1_ТАБ1 SKPMAME010, SW20_Б1 SKPMAME010, SW21_Й1 SKPMAME010, SW22_Р1 SKPMAME010, SW23_З1 SKPMAME010, SW24_AP2 SKPMAME010, SW25_ЗБ1 SKPMAME010, SW26_3 SKPMAME010, SW27_;1 SKPMAME010, SW28_Ц1 SKPMAME010, SW29_К1 SKPMAME010, SW2_0 SKPMAME010, SW30_С1 SKPMAME010, SW31_Ш1 SKPMAME010, SW32_F1 SKPMAME010, SW33_LT1 SKPMAME010, SW34_4 SKPMAME010, SW35 SKPMAME010, SW36_Д1 SKPMAME010, SW37_Л1 SKPMAME010, SW38_Т1 SKPMAME010, SW39_Э1 SKPMAME010, SW3_8 SKPMAME010, SW40_F2 SKPMAME010, SW41_UP1 SKPMAME010, SW42_5 SKPMAME010, SW43_-=1 SKPMAME010, SW44_E1 SKPMAME010, SW45_М1 SKPMAME010, SW46_У1 SKPMAME010, SW47_Щ1 SKPMAME010, SW48_F3 SKPMAME010, SW49_RT1 SKPMAME010, SW4_Ю1 SKPMAME010, SW50_6 SKPMAME010, SW51 SKPMAME010, SW52_Ф1 SKPMAME010, SW53_Н1 SKPMAME010, SW54_Ж1 SKPMAME010, SW55_Ч1 SKPMAME010, SW56_F4 SKPMAME010, SW57_DN1 SKPMAME010, SW58_7 SKPMAME010, SW59_/1 SKPMAME010, SW5_Х1 SKPMAME010, SW60_Г1 SKPMAME010, SW61_О1 SKPMAME010, SW62_В1 SKPMAME010, SW63_SPC1 SKPMAME010, SW63_SPC2 SKPMAME010, SW64_F5 SKPMAME010, SW6_П1 SKPMAME010, SW7_Ь1 SKPMAME010, SW8_HOME1 SKPMAME010, SW9_ПС1 SKPMAME010, U1 Pico

Commit message: readme lala
Parts:
- added D12: BAT54S, Package_TO_SOT_SMD:SOT-23, symbol Diode:BAT54S
Connections:
- net VSYS: now also D12.3 (COM); no longer U1.39 (VSYS)
- new net VSYSx: D12.2 (K), U1.39 (VSYS)
- no-connect marks 0 -> 1
Changed lines of the file:
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@@
   (junction (at 278.13 138.43) (diameter 0) (color 0 0 0 0)
   )
+  (no_connect (at 189.23 208.28))
   (wire (pts (xy 115.57 134.62) (xy 115.57 147.32))
     (stroke (width 0) (type default))
@@
   )
   (wire (pts (xy 173.99 100.33) (xy 182.88 100.33))
+    (stroke (width 0) (type default))
+  )
+  (wire (pts (xy 181.61 203.2) (xy 189.23 203.2))
     (stroke (width 0) (type default))
   )
@@
     (effects (font (size 1.27 1.27)) (justify right bottom))
   )
+  (label "VSYSx" (at 170.18 208.28 180) (fields_autoplaced)
+    (effects (font (size 1.27 1.27)) (justify right bottom))
+  )
   (label "~{ИНД \"РУС\"}" (at 63.5 130.81 180) (fields_autoplaced)
     (effects (font (size 1.27 1.27)) (justify right bottom))
@@
     (effects (font (size 1.27 1.27)) (justify left bottom))
   )
-  (label "VSYS" (at 173.99 208.28 180) (fields_autoplaced)
+  (label "VSYS" (at 189.23 203.2 180) (fields_autoplaced)
     (effects (font (size 1.27 1.27)) (justify right bottom))
   )
@@
         )
       )
+    )
+  )
+  (symbol (lib_id "Diode:BAT54S") (at 181.61 208.28 180) (unit 1)
+    (in_bom yes) (on_board yes) (dnp no) (fields_autoplaced)
+    (property "Reference" "D12" (at 181.61 212.09 0)
+      (effects (font (size 1.27 1.27)))
+    )
+    (property "Value" "BAT54S" (at 181.61 214.63 0)
+      (effects (font (size 1.27 1.27)))
+    )
+    (property "Footprint" "Package_TO_SOT_SMD:SOT-23" (at 179.705 211.455 0)
+      (effects (font (size 1.27 1.27)) (justify left) hide)
+    )
+    (property "Datasheet" "https://www.diodes.com/assets/Datasheets/ds11005.pdf" (at 184.658 208.28 0)
+      (effects (font (size 1.27 1.27)) hide)
+    )
+    (pin "1")
+    (pin "2")
+    (pin "3")
+    (instances
+      (project "v06ckeyboard"
+        (path "/d5f54b25-d4a8-4887-bfd2-29d51dc4b499"
+          (reference "D12") (unit 1)
+        )
+      )
